Commit message: Update Sidewinder URDF

File: sidewinder_description/urdf/sidewinder.urdf (robot description, URDF)
Before this commit: robot sidewinder, 4 links, 3 joints
Joints:
- joint joint2: origin xyz=-0.1016 -0.17598 0 -> xyz=-0.1016 0.17598 0
- joint joint3: origin xyz=-0.1016 0.17598 0 -> xyz=-0.1016 -0.17598 0
